File: Board/Board.kicad_pcb (KiCad board)
At the start: 2 copper layers, 0 parts

Commit message: built power circuit
Parts:
- added C1: 100nF, Capacitor_SMD:C_0805_2012Metric_Pad1.15x1.40mm_HandSolder, F.Cu at (73.0, 91.1)
- added C2: 100nF, Capacitor_SMD:C_0805_2012Metric_Pad1.15x1.40mm_HandSolder, F.Cu at (84.3, 88.0)
- added C3: 100nF, Capacitor_SMD:C_0805_2012Metric_Pad1.15x1.40mm_HandSolder, F.Cu at (77.7, 91.1)
- added C4: 10nF, Capacitor_SMD:C_0805_2012Metric_Pad1.15x1.40mm_HandSolder, F.Cu at (92.7, 74.9)
- added C5: 10nF, Capacitor_SMD:C_0805_2012Metric_Pad1.15x1.40mm_HandSolder, F.Cu at (82.5, 91.1)
- added C6: 100nF, Capacitor_SMD:C_0805_2012Metric_Pad1.15x1.40mm_HandSolder, F.Cu at (89.1, 88.0)
- added C7: 100nF, Capacitor_SMD:C_0805_2012Metric_Pad1.15x1.40mm_HandSolder, F.Cu at (92.7, 78.7)
- added C8: 10nF, Capacitor_SMD:C_0805_2012Metric_Pad1.15x1.40mm_HandSolder, F.Cu at (87.2, 90.9)
- added C9: 100nF, Capacitor_SMD:C_0805_2012Metric_Pad1.15x1.40mm_HandSolder, F.Cu at (94.2, 85.6)
- added Q1: Q_PNP_BCEC, Package_TO_SOT_SMD:SOT-223, F.Cu at (82.5, 76.2)
- added R1: 1k00, Resistor_SMD:R_0805_2012Metric_Pad1.15x1.40mm_HandSolder, F.Cu at (83.8, 83.8)
- added U1: ADAU1701, Package_QFP:LQFP-48_7x7mm_P0.5mm, F.Cu at (68.6, 77.5)
