File: Board/Board.kicad_pcb (KiCad board)
At the start: 2 copper layers, 100 x 100 mm, 75 parts, among them J1 MP 0-2, J2 Audio In, J3 MP 3-5, J4 MP 6-8, J5 MP 9-11, J6 Power Connector, J7 Audio Out (Headphones), J8 CONN_EEPROM, Q1 Q_PNP_BCEC, U1 ADAU1701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

Commit message: done
Parts:
- added C39: .22uF, Capacitor_SMD:C_0805_2012Metric_Pad1.15x1.40mm_HandSolder, F.Cu at (85.1, -19.7)
- added C40: .22uF, Capacitor_SMD:C_0805_2012Metric_Pad1.15x1.40mm_HandSolder, F.Cu at (93.5, -28.1)
- added C41: .22uF, Capacitor_SMD:C_0805_2012Metric_Pad1.15x1.40mm_HandSolder, F.Cu at (85.1, -16.8)
- added C42: .22uF, Capacitor_SMD:C_0805_2012Metric_Pad1.15x1.40mm_HandSolder, F.Cu at (148.5, -53.7)
- added C43: .22uF, Capacitor_SMD:C_0805_2012Metric_Pad1.15x1.40mm_HandSolder, F.Cu at (153.2, -56.7)
- added C44: .22uF, Capacitor_SMD:C_0805_2012Metric_Pad1.15x1.40mm_HandSolder, F.Cu at (156.9, -62.1)
- added C45: .22uF, Capacitor_SMD:C_0805_2012Metric_Pad1.15x1.40mm_HandSolder, F.Cu at (161.6, -65.1)
- added C6: .22uF, Capacitor_SMD:C_0805_2012Metric_Pad1.15x1.40mm_HandSolder, F.Cu at (85.1, -10.9)
- added J10: NOT_PWR_CONN, Connector_PinHeader_2.54mm:PinHeader_1x01_P2.54mm_Vertical, F.Cu at (107.0, -64.2)
- added J11: 3.3V_Conn, Connector_PinHeader_2.54mm:PinHeader_1x01_P2.54mm_Vertical, F.Cu at (77.3, -38.5)
- added J12: GND_Conn, Connector_PinHeader_2.54mm:PinHeader_1x01_P2.54mm_Vertical, F.Cu at (81.9, -44.4)
- added J13: 5V_Conn, Connector_PinHeader_2.54mm:PinHeader_1x01_P2.54mm_Vertical, F.Cu at (86.6, -42.9)
- added J14: THERM, Connector_PinHeader_2.54mm:PinHeader_1x01_P2.54mm_Vertical, F.Cu at (94.6, -18.4)
- added J15: Gain_Conn, Connector_PinHeader_2.54mm:PinHeader_1x01_P2.54mm_Vertical, F.Cu at (99.3, -21.4)
- added J16: THERM, Connector_PinHeader_2.54mm:PinHeader_1x01_P2.54mm_Vertical, F.Cu at (157.9, -55.4)
- added J17: Gain_Conn, Connector_PinHeader_2.54mm:PinHeader_1x01_P2.54mm_Vertical, F.Cu at (162.7, -58.3)
- added J9: Conn_01x03_Female, 691213710003:691213710003, F.Cu at (137.8, -51.7)
- J1: value MP 0-2 -> Conn_01x03_Female
- J2: value Audio In -> Conn_01x03_Female
- J3: value MP 3-5 -> Conn_01x12_Female; footprint 691213710003:691213710003 -> Connector_PinHeader_2.54mm:PinHeader_1x12_P2.54mm_Vertical
- J4: value MP 6-8 -> Conn_01x03_Female
- J5: value MP 9-11 -> Conn_01x03_Female
- J6: value Power Connector -> Conn_01x03_Female
- J7: value Audio Out (Headphones) -> Conn_01x03_Female
- S1: footprint Switch:JS202011SCQN -> Switch JS202011SCQN:SW_JS202011SCQN
- U5: footprint CAT24 EEPROM:CAT24C16WI-GT3 -> CAT24:CAT24C16WI-GT3
- moved R5 189.3 mm to (122.1, -25.2)
- moved C11 188.1 mm to (112.3, -9.89)
- moved R12 184.0 mm to (112.3, -12.8)
- moved R6 184.0 mm to (107.5, -9.89)
- moved R16 182.7 mm to (89.9, -13.8)
- moved R22 182.5 mm to (141.4, -41.5)
- moved C12 182.4 mm to (117.0, -12.8)
- moved C10 182.2 mm to (117.4, -25.2)
- moved C3 182.2 mm to (121.8, -19.3)
- moved C33 182.2 mm to (112.3, -19.9)
- moved C34 182.2 mm to (117.4, -28.1)
- moved C4 182.2 mm to (122.1, -22.2)
- moved C5 182.2 mm to (117.0, -19.3)
- moved C8 182.2 mm to (117.4, -22.2)
- moved C9 182.2 mm to (122.1, -28.1)
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Connections:
- J1 pad 1: Net-(J1-Pad1) -> GND
- J2 pad 1: Net-(J2-Pad1) -> GND
- J2 pad 2: Net-(J2-Pad2) -> GND
- J2 pad 3: Net-(J2-Pad3) -> +12V
- J4 pad 1: Net-(J4-Pad1) -> /SSM3302_1/IN_R
- J4 pad 2: Net-(J4-Pad2) -> /SSM3302_1/IN_L
- J4 pad 3: Net-(J4-Pad3) -> GND
- J5 pad 1: Net-(J5-Pad1) -> Net-(C39-Pad2)
- J5 pad 2: Net-(J5-Pad2) -> Net-(C6-Pad2)
- J5 pad 3: Net-(J5-Pad3) -> Net-(C6-Pad2)
- J6 pad 1: GND -> Net-(C40-Pad1)
- J6 pad 2: GND -> Net-(C40-Pad1)
- J6 pad 3: +12V -> Net-(C41-Pad1)
- J7 pad 1: /SSM3302_1/IN_R -> Net-(C43-Pad2)
- J7 pad 2: /SSM3302_1/IN_L -> Net-(C42-Pad2)
- J7 pad 3: GND -> Net-(C42-Pad2)
- R2 pad 2: Net-(R2-Pad2) -> Net-(J1-Pad3)
- R3 pad 2: Net-(R3-Pad2) -> Net-(J1-Pad2)
- U1 pad 10: Net-(J1-Pad2) -> Net-(J3-Pad2)
- U1 pad 11: Net-(J1-Pad1) -> Net-(J3-Pad1)
- U1 pad 14: Net-(J4-Pad2) -> Net-(J3-Pad8)
- U1 pad 15: Net-(J4-Pad1) -> Net-(J3-Pad7)
- U1 pad 16: Net-(J5-Pad2) -> Net-(J3-Pad11)
- U1 pad 19: Net-(J5-Pad3) -> Net-(J3-Pad12)
- U1 pad 26: Net-(J5-Pad1) -> Net-(J3-Pad10)
- U1 pad 27: Net-(J4-Pad3) -> Net-(J3-Pad9)
- U1 pad 28: Net-(J3-Pad1) -> Net-(J3-Pad4)
- U1 pad 29: Net-(J1-Pad3) -> Net-(J3-Pad3)
- U1 pad 8: Net-(J3-Pad2) -> Net-(J3-Pad5)
- U1 pad 9: Net-(J3-Pad3) -> Net-(J3-Pad6)
- U2 pad 10: Net-(U2-Pad10) -> +5V
- U2 pad 11: Net-(R16-Pad1) -> /SSM3302_1/IN_L
- U2 pad 12: /SSM3302_1/IN_L -> Net-(R16-Pad1)
- U2 pad 14: Net-(U2-Pad14) -> GND
- U2 pad 15: Net-(U2-Pad15) -> GND
- U2 pad 16: Net-(U2-Pad16) -> GND
- U2 pad 2: Net-(U2-Pad2) -> Net-(C6-Pad2)
- U2 pad 22: Net-(U2-Pad22) -> NOT_PWR
- U2 pad 23: Net-(U2-Pad23) -> +3V3
- U2 pad 24: Net-(U2-Pad24) -> GND
- U2 pad 26: Net-(U2-Pad26) -> Net-(C41-Pad1)
- U2 pad 27: Net-(U2-Pad27) -> Net-(C41-Pad1)
- U2 pad 28: Net-(U2-Pad28) -> Net-(C40-Pad1)
- U2 pad 29: Net-(U2-Pad29) -> Net-(C40-Pad1)
- U2 pad 3: Net-(U2-Pad3) -> Net-(C6-Pad2)
- U2 pad 4: Net-(U2-Pad4) -> Net-(C39-Pad2)
- U2 pad 5: Net-(U2-Pad5) -> Net-(C39-Pad2)
- U2 pad 7: Net-(U2-Pad7) -> GND
- U2 pad 8: Net-(U2-Pad8) -> +5V
- U2 pad 9: Net-(U2-Pad9) -> NOT_PWR
- U2 pad HTAB: Net-(U2-PadHTAB) -> GND
- U4 pad 10: Net-(U4-Pad10) -> +5V
- U4 pad 11: Net-(R18-Pad1) -> /SSM3302_2/IN_L
- U4 pad 12: /SSM3302_2/IN_L -> Net-(R18-Pad1)
- U4 pad 14: Net-(U4-Pad14) -> GND
- U4 pad 15: Net-(U4-Pad15) -> GND
- U4 pad 16: Net-(U4-Pad16) -> GND
- U4 pad 2: Net-(U4-Pad2) -> Net-(C42-Pad2)
- U4 pad 22: Net-(U4-Pad22) -> NOT_PWR
- U4 pad 23: Net-(U4-Pad23) -> +3V3
- U4 pad 24: Net-(U4-Pad24) -> GND
- U4 pad 26: Net-(U4-Pad26) -> Net-(C45-Pad1)
- U4 pad 27: Net-(U4-Pad27) -> Net-(C45-Pad1)
- U4 pad 28: Net-(U4-Pad28) -> Net-(C44-Pad1)
- U4 pad 29: Net-(U4-Pad29) -> Net-(C44-Pad1)
- U4 pad 3: Net-(U4-Pad3) -> Net-(C42-Pad2)
- U4 pad 4: Net-(U4-Pad4) -> Net-(C43-Pad2)
- U4 pad 5: Net-(U4-Pad5) -> Net-(C43-Pad2)
- U4 pad 7: Net-(U4-Pad7) -> GND
- U4 pad 8: Net-(U4-Pad8) -> +5V
- U4 pad 9: Net-(U4-Pad9) -> NOT_PWR
- U4 pad HTAB: Net-(U4-PadHTAB) -> GND

Commit message: split
Parts:
- removed J13: 5V_Conn, Connector_PinHeader_2.54mm:PinHeader_1x01_P2.54mm_Vertical
- added C46: 56nF, Capacitor_SMD:C_0805_2012Metric_Pad1.15x1.40mm_HandSolder, F.Cu at (116.5, -94.4)
- added C47: 3n3F, Capacitor_SMD:C_0805_2012Metric_Pad1.15x1.40mm_HandSolder, F.Cu at (124.1, -102.7)
- added C48: 100nF, Capacitor_SMD:C_0805_2012Metric_Pad1.15x1.40mm_HandSolder, F.Cu at (104.9, -84.4)
- added C49: 10uF, Capacitor_SMD:C_0805_2012Metric_Pad1.15x1.40mm_HandSolder, F.Cu at (111.3, -90.6)
- added C50: 100nF, Capacitor_SMD:C_0805_2012Metric_Pad1.15x1.40mm_HandSolder, F.Cu at (124.1, -105.6)
- added C51: 10uF, Capacitor_SMD:C_0805_2012Metric_Pad1.15x1.40mm_HandSolder, F.Cu at (116.5, -97.4)
- added C52: 100nF, Capacitor_SMD:C_0805_2012Metric_Pad1.15x1.40mm_HandSolder, F.Cu at (121.3, -97.4)
- added C53: 47uF, Capacitor_SMD:C_0805_2012Metric_Pad1.15x1.40mm_HandSolder, F.Cu at (106.5, -87.3)
- added J18: WB_Pin, Connector_PinHeader_2.54mm:PinHeader_1x01_P2.54mm_Vertical, F.Cu at (126.0, -97.2)
- added J19: Reset, Connector_PinHeader_2.54mm:PinHeader_1x01_P2.54mm_Vertical, F.Cu at (109.6, -83.5)
- added R23: 475r, Resistor_SMD:R_0805_2012Metric_Pad1.15x1.40mm_HandSolder, F.Cu at (107.0, -93.5)
- C10, C8: value 100nF -> 10uF
- C13, C15, C17, C19: value 5n6F -> 4.7nF
- C24, C25: value 1uF -> 100nF
- C33, C34: value 100nF -> 1uF
- C5, C9: value 10uF -> 100nF
- J5, J6, J7, J9: value Conn_01x03_Female -> Conn_01x02_Female; footprint 691213710003:691213710003 -> WJ250A-3.50-2P:WJ250A3502P
- R10: value 140k -> 2k20
- R11: value 78.7k -> 2k20
- R20: value 2k20 -> 1k00
- R21: value 2k20 -> 140k
- R22: value 2k20 -> 78.7k
- R4: value 100 -> 2k20
- R5: value 1k00 -> 100
- U3: value ADP3336ARMZ -> CAT24C16WI-GT3; footprint Package_SO:MSOP-8_3x3mm_P0.65mm -> CAT24:CAT24C16WI-GT3
- U5: value CAT24C16WI-GT3 -> ADP3336ARMZ; footprint CAT24:CAT24C16WI-GT3 -> Package_SO:MSOP-8_3x3mm_P0.65mm
- Y1: footprint ECS-122.8-20-3X-EN-TR:XTAL_ECS-122.8-20-3X-EN-TR -> 5032_2P:OSCCC500X320X135
- moved J7 201.7 mm to (100.6, 136.6)
- moved C45 196.7 mm to (132.6, 129.4)
- moved C30 195.4 mm to (123.0, 129.4)
- moved C44 194.0 mm to (144.1, 131.5)
- moved C38 190.4 mm to (133.5, 123.9)
- moved J9 190.0 mm to (112.4, 136.6)
- moved C37 188.2 mm to (144.1, 128.5)
- moved C43 186.8 mm to (137.3, 129.4)
- moved U4 185.3 mm to (145.9, 122.9)
- moved J16 185.0 mm to (148.8, 129.4)
- moved R18 183.0 mm to (119.2, 123.9)
- moved J17 182.6 mm to (152.4, 124.0)
- moved C32 181.4 mm to (127.8, 129.4)
- moved C17 181.3 mm to (100.6, 109.9)
- moved C31 179.4 mm to (128.7, 123.9)
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Connections:
- net /oscillator/MCLKI renamed Net-(C2-Pad2)
- net NOT_PWR renamed /SSM3302_1/AMP_PWR
- C10 pad 2: /power/DVDD -> Net-(C10-Pad2)
- C24 pad 1: +12V -> GND
- C24 pad 2: GND -> Net-(C10-Pad2)
- C25 pad 1: +3V3 -> GND
- C25 pad 2: GND -> Net-(C10-Pad2)
- C33 pad 1: +3V3 -> +12V
- C34 pad 1: GND -> +3V3
- C34 pad 2: /power/DVDD -> GND
- C7 pad 1: GND -> +3V3
- C7 pad 2: +3V3 -> GND
- C9 pad 2: /power/DVDD -> +3V3
- J5 pad 1: Net-(C39-Pad2) -> Net-(C43-Pad2)
- J5 pad 2: Net-(C6-Pad2) -> Net-(C42-Pad2)
- J6 pad 1: Net-(C40-Pad1) -> Net-(C44-Pad1)
- J6 pad 2: Net-(C40-Pad1) -> Net-(C45-Pad1)
- J7 pad 1: Net-(C43-Pad2) -> Net-(C39-Pad2)
- J7 pad 2: Net-(C42-Pad2) -> Net-(C6-Pad2)
- J8 pad 1: /EEPROM/SCL -> Net-(J8-Pad1)
- J8 pad 2: /EEPROM/SDA -> Net-(J8-Pad2)
- J9 pad 1: Net-(C44-Pad1) -> Net-(C40-Pad1)
- J9 pad 2: Net-(C44-Pad1) -> Net-(C41-Pad1)
- Q1 pad 1: /power/VDRIVE -> Net-(Q1-Pad1)
- Q1 pad 2: /power/DVDD -> Net-(C10-Pad2)
- Q1 pad 4: /power/DVDD -> Net-(C10-Pad2)
- R1 pad 1: Net-(R1-Pad1) -> GND
- R1 pad 2: GND -> Net-(R1-Pad2)
- R10 pad 2: Net-(R10-Pad2) -> Net-(J8-Pad2)
- R11 pad 1: Net-(R10-Pad2) -> +3V3
- R11 pad 2: GND -> Net-(R11-Pad2)
- R20 pad 2: /EEPROM/SCL -> Net-(Q1-Pad1)
- R21 pad 2: /EEPROM/SDA -> Net-(R21-Pad2)
- R22 pad 1: +3V3 -> Net-(R21-Pad2)
- R22 pad 2: Net-(R22-Pad2) -> GND
- R4 pad 1: /oscillator/OSCO -> +3V3
- R4 pad 2: Net-(C1-Pad2) -> Net-(J8-Pad1)
- R5 pad 1: +3V3 -> Net-(R5-Pad1)
- R5 pad 2: /power/VDRIVE -> Net-(C1-Pad2)
- S1 pad 2: /EEPROM/WP -> Net-(S1-Pad2)
- S1 pad 3: Net-(R22-Pad2) -> Net-(S1-Pad3)
- S1 pad 4: GND -> Net-(S1-Pad4)
- S1 pad 5: /EEPROM/WP -> Net-(S1-Pad5)
- S1 pad 6: Net-(R22-Pad2) -> Net-(R11-Pad2)
- U1 pad 13: /power/DVDD -> Net-(C10-Pad2)
- U1 pad 17: /power/VDRIVE -> Net-(Q1-Pad1)
- U1 pad 21: /EEPROM/WP -> Net-(S1-Pad5)
- U1 pad 22: /EEPROM/SDA -> Net-(J8-Pad2)
- U1 pad 23: /EEPROM/SCL -> Net-(J8-Pad1)
- U1 pad 24: /power/DVDD -> Net-(C10-Pad2)
- U1 pad 3: Net-(R1-Pad1) -> Net-(R1-Pad2)
- U1 pad 31: /oscillator/OSCO -> Net-(R5-Pad1)
- U1 pad 38: Net-(U1-Pad38) -> GND
- U1 pad 39: Net-(U1-Pad39) -> +3V3
- U1 pad 6: Net-(U1-Pad6) -> +3V3
- U1 pad 7: Net-(U1-Pad7) -> GND
- U3 pad 1: +3V3 -> Net-(U3-Pad1)
- U3 pad 2: +3V3 -> Net-(U3-Pad2)
- U3 pad 3: +3V3 -> Net-(U3-Pad3)
- U3 pad 5: Net-(R10-Pad2) -> Net-(J8-Pad2)
- U3 pad 6: +12V -> Net-(J8-Pad1)
- U3 pad 7: +12V -> Net-(S1-Pad5)
- U3 pad 8: +12V -> +3V3
- U5 pad 1: Net-(U5-Pad1) -> +3V3
- U5 pad 2: Net-(U5-Pad2) -> +3V3
- U5 pad 3: Net-(U5-Pad3) -> +3V3
- U5 pad 5: /EEPROM/SDA -> Net-(R21-Pad2)
- U5 pad 6: /EEPROM/SCL -> +12V
- U5 pad 7: /EEPROM/WP -> +12V
- U5 pad 8: +3V3 -> +12V
