File: Board/ADP3336.sch (KiCad schematic (older format))
At the start: 5 parts, among them U3 ADP3336ARMZ

Commit message: did some more stuff
Parts:
- C24, C25: footprint (none) -> Capacitor_SMD:C_0805_2012Metric_Pad1.15x1.40mm_HandSolder
Changed lines of the file:
@@
 EESchema Schematic File Version 4
+LIBS:Board-cache
 EELAYER 30 0
 EELAYER END
 $Descr A4 11693 8268
 encoding utf-8
-Sheet 9 9
+Sheet 9 12
 Title ""
 Date ""
@@
 F 0 "C24" H 4400 3850 50  0000 L CNN
 F 1 "1uF" H 4350 3750 50  0000 L CNN
-F 2 "" H 4600 3800 50  0001 C CNN
+F 2 "Capacitor_SMD:C_0805_2012Metric_Pad1.15x1.40mm_HandSolder" H 4600 3800 50  0001 C CNN
 F 3 "~" H 4600 3800 50  0001 C CNN
 	1    4600 3800
@@
 F 0 "C25" H 6492 3696 50  0000 L CNN
 F 1 "1uF" H 6492 3605 50  0000 L CNN
-F 2 "" H 6400 3650 50  0001 C CNN
+F 2 "Capacitor_SMD:C_0805_2012Metric_Pad1.15x1.40mm_HandSolder" H 6400 3650 50  0001 C CNN
 F 3 "~" H 6400 3650 50  0001 C CNN
 	1    6400 3650
