File: Board/power.sch (KiCad schematic (older format))
At the start: 11 parts, among them Q1 Q_PNP_BCEC

Commit message: more improvements
Connections:
- net VDD renamed +3V3
Changed lines of the file:
@@
 $Descr A4 11693 8268
 encoding utf-8
-Sheet 3 3
+Sheet 3 9
 Title ""
 Date ""
@@
 Comment4 ""
 $EndDescr
-$Comp
-L power:VDD #PWR?
-U 1 1 5DE1F53E
-P 5100 2700
-AR Path="/5DE1F53E" Ref="#PWR?"  Part="1"
-AR Path="/5DE1C9A6/5DE1F53E" Ref="#PWR0103"  Part="1"
-F 0 "#PWR0103" H 5100 2550 50  0001 C CNN
-F 1 "VDD" H 5117 2873 50  0000 C CNN
-F 2 "" H 5100 2700 50  0001 C CNN
-F 3 "" H 5100 2700 50  0001 C CNN
-	1    5100 2700
-	1    0    0    -1
-$EndComp
 $Comp
 L Device:C_Small C?
@@
 Wire Wire Line
 	4400 4000 4400 3650
-$Comp
-L power:VDD #PWR?
-U 1 1 5DE1F580
-P 6950 4100
-AR Path="/5DE1F580" Ref="#PWR?"  Part="1"
-AR Path="/5DE1C9A6/5DE1F580" Ref="#PWR0105"  Part="1"
-F 0 "#PWR0105" H 6950 3950 50  0001 C CNN
-F 1 "VDD" H 6967 4273 50  0000 C CNN
-F 2 "" H 6950 4100 50  0001 C CNN
-F 3 "" H 6950 4100 50  0001 C CNN
-	1    6950 4100
-	1    0    0    -1
-$EndComp
 Wire Wire Line
 	6050 3300 6300 3300
@@
 	6500 5000 6950 5000
 Connection ~ 6950 5000
+$Comp
+L power:+3.3V #PWR0114
+U 1 1 5DEBD049
+P 5100 2700
+F 0 "#PWR0114" H 5100 2550 50  0001 C CNN
+F 1 "+3.3V" H 5115 2873 50  0000 C CNN
+F 2 "" H 5100 2700 50  0001 C CNN
+F 3 "" H 5100 2700 50  0001 C CNN
+	1    5100 2700
+	1    0    0    -1
+$EndComp
+$Comp
+L power:+3.3V #PWR0115
+U 1 1 5DEBE65C
+P 6950 4100
+F 0 "#PWR0115" H 6950 3950 50  0001 C CNN
+F 1 "+3.3V" H 6965 4273 50  0000 C CNN
+F 2 "" H 6950 4100 50  0001 C CNN
+F 3 "" H 6950 4100 50  0001 C CNN
+	1    6950 4100
+	1    0    0    -1
+$EndComp
 $EndSCHEMATC

Commit message: did some more stuff
Parts:
- removed C11: 100nF, Capacitor_SMD:C_0805_2012Metric_Pad1.15x1.40mm_HandSolder, symbol Device:C_Small
- removed C6: 10nF, Capacitor_SMD:C_0805_2012Metric_Pad1.15x1.40mm_HandSolder, symbol Device:C_Small
- added C33, C34: 100nF, Capacitor_SMD:C_0805_2012Metric_Pad1.15x1.40mm_HandSolder, symbol Device:C_Small
- C5: value 100nF -> 10uF
- C7, C9: value 10nF -> 10uF
Connections:
- net +3V3: now also C33.1
- net DVDD: now also C34.2
- net GND: now also C33.2, C34.1
Other:
- moved on the sheet: C10, C3, C4, C5, C9
