File: Board/Board.sch (KiCad schematic (older format))
At the start: 13 parts, among them J1 Conn_01x12_Female, Q1 Q_PNP_BCEC, U1 ADAU1701

Commit message: did some more stuff
Parts:
- removed C1, C2, C3, C6, C7, C9: 100nF, Capacitor_SMD:C_0805_2012Metric_Pad1.15x1.40mm_HandSolder, symbol Device:C_Small
- removed C4, C5, C8: 10nF, Capacitor_SMD:C_0805_2012Metric_Pad1.15x1.40mm_HandSolder, symbol Device:C_Small
- removed J1: Conn_01x12_Female, Connector_PinSocket_2.54mm:PinSocket_1x12_P2.54mm_Vertical, symbol Connector:Conn_01x12_Female
- removed Q1: Q_PNP_BCEC, Package_TO_SOT_SMD:SOT-223, symbol Device:Q_PNP_BCEC
- added J1: Conn_01x12_Male, Connector_Phoenix_MSTB:PhoenixContact_MSTBVA_2,5_12-G_1x12_P5.00mm_Vertical, symbol Connector:Conn_01x12_Male
- added J2: Audio In, Connector_Phoenix_MSTB:PhoenixContact_MSTBA_2,5_3-G_1x03_P5.00mm_Horizontal, symbol Connector:Conn_01x03_Male
- added R2, R3: 18k0, Resistor_SMD:R_0805_2012Metric_Pad1.15x1.40mm_HandSolder, symbol Device:R_Small_US
- R1: value 1k00 -> 18k
Connections:
- net labels removed: VDD
- wire segments 70 -> 43

Commit message: more improvements
Parts:
- removed J1: Conn_01x12_Male, Connector_Phoenix_MSTB:PhoenixContact_MSTBVA_2,5_12-G_1x12_P5.00mm_Vertical, symbol Connector:Conn_01x12_Male
- added J1: MP 0-2, 691213710003:691213710003, symbol Connector:Conn_01x03_Male
- added J3: MP 3-5, 691213710003:691213710003, symbol Connector:Conn_01x03_Male
- added J4: MP 6-8, 691213710003:691213710003, symbol Connector:Conn_01x03_Male
- added J5: MP 9-11, 691213710003:691213710003, symbol Connector:Conn_01x03_Male
- added J6: Power Connector, 691213710003:691213710003, symbol Connector:Conn_01x03_Male
- added J7: Audio Out (Headphones), 691213710003:691213710003, symbol Connector:Conn_01x03_Male
- J2: footprint Connector_Phoenix_MSTB:PhoenixContact_MSTBA_2,5_3-G_1x03_P5.00mm_Horizontal -> 691213710003:691213710003
Connections:
- net labels added: +12V
- wire segments 43 -> 76
Other:
- moved on the sheet: J2, R1, R2, R3, U1

Commit message: did some more stuff
Parts:
- added J8: CONN_EEPROM, Connector_PinHeader_2.54mm:PinHeader_1x02_P2.54mm_Vertical, symbol Connector:Conn_01x02_Female
Connections:
- net labels added: +3.3V
- wire segments 76 -> 95
Other:
- moved on the sheet: J6
Changed lines of the file:
@@
 EESchema Schematic File Version 4
+LIBS:Board-cache
 EELAYER 30 0
 EELAYER END
 $Descr A4 11693 8268
 encoding utf-8
-Sheet 1 9
+Sheet 1 12
 Title ""
 Date ""
@@
 	4400 2850 5400 2850
 Wire Wire Line
-	4950 2700 6450 2700
-Wire Wire Line
-	5900 2900 6450 2900
-Wire Wire Line
 	4950 2350 6200 2350
 $Comp
@@
 F0 "SSM3302_1" 50
 F1 "SSM3302.sch" 50
-$EndSheet
-$Sheet
-S 5450 1200 700  550
+F2 "IN_L" I L 7050 2650 50
+F3 "IN_R" I L 7050 2500 50
+$EndSheet
+$Sheet
+S 5300 800  700  550
 U 5DEA6AA8
 F0 "ADP3336" 50
 F1 "ADP3336.sch" 50
-F2 "12V_in" I L 5450 1350 50
-F3 "3.3V_out" O R 6150 1600 50
+F2 "12V_in" I L 5300 950 50
+F3 "3.3V_out" O R 6000 1150 50
 $EndSheet
 $Comp
 L power:+12V #PWR0103
 U 1 1 5DEB2FF5
-P 4950 1050
-F 0 "#PWR0103" H 4950 900 50  0001 C CNN
-F 1 "+12V" H 4965 1223 50  0000 C CNN
-F 2 "" H 4950 1050 50  0001 C CNN
-F 3 "" H 4950 1050 50  0001 C CNN
-	1    4950 1050
+P 4800 900
+F 0 "#PWR0103" H 4800 750 50  0001 C CNN
+F 1 "+12V" H 4815 1073 50  0000 C CNN
+F 2 "" H 4800 900 50  0001 C CNN
+F 3 "" H 4800 900 50  0001 C CNN
+	1    4800 900
 	1    0    0    -1
 $EndComp
@@
 L Connector:Conn_01x03_Male J6
 U 1 1 5DEB3305
-P 4600 1200
-F 0 "J6" H 4692 875 50  0000 C CNN
-F 1 "Power Connector" H 4692 966 50  0000 C CNN
-F 2 "691213710003:691213710003" H 4800 1200 50  0001 C CNN
-F 3 "~" H 4800 1200 50  0001 C CNN
-	1    4600 1200
+P 4450 1050
+F 0 "J6" H 4542 725 50  0000 C CNN
+F 1 "Power Connector" H 4542 816 50  0000 C CNN
+F 2 "691213710003:691213710003" H 4650 1050 50  0001 C CNN
+F 3 "~" H 4650 1050 50  0001 C CNN
+	1    4450 1050
 	-1   0    0    1
 $EndComp
 Wire Wire Line
-	4600 1100 4950 1100
-Wire Wire Line
-	4950 1100 4950 1050
-Wire Wire Line
-	4950 1100 5250 1100
-Wire Wire Line
-	5250 1100 5250 1350
-Wire Wire Line
-	5250 1350 5450 1350
-Connection ~ 4950 1100
-Wire Wire Line
-	4600 1200 4700 1200
-Wire Wire Line
-	4700 1200 4700 1300
-Wire Wire Line
-	4700 1300 4600 1300
-Wire Wire Line
-	4700 1300 4700 1450
-Connection ~ 4700 1300
+	4450 950  4800 950
+Wire Wire Line
+	4800 950  4800 900
+Connection ~ 4800 950
+Wire Wire Line
+	4450 1050 4550 1050
+Wire Wire Line
+	4550 1050 4550 1150
+Wire Wire Line
+	4550 1150 4450 1150
+Wire Wire Line
+	4550 1150 4550 1300
+Connection ~ 4550 1150
 $Comp
 L power:GND #PWR0105
 U 1 1 5DEBBA8D
-P 4700 1450
-F 0 "#PWR0105" H 4700 1200 50  0001 C CNN
-F 1 "GND" H 4705 1277 50  0000 C CNN
-F 2 "" H 4700 1450 50  0001 C CNN
-F 3 "" H 4700 1450 50  0001 C CNN
-	1    4700 1450
+P 4550 1300
+F 0 "#PWR0105" H 4550 1050 50  0001 C CNN
+F 1 "GND" H 4555 1127 50  0000 C CNN
+F 2 "" H 4550 1300 50  0001 C CNN
+F 3 "" H 4550 1300 50  0001 C CNN
+	1    4550 1300
 	1    0    0    -1
 $EndComp
@@
 Connection ~ 6300 2550
 Wire Wire Line
-	6300 2550 6450 2550
-Wire Wire Line
 	6550 1800 6200 1800
 Wire Wire Line
@@
 Connection ~ 6200 2350
 Wire Wire Line
-	6200 2350 6450 2350
+	4800 950  5300 950
+$Comp
+L power:+3.3V #PWR0124
+U 1 1 5DEE7D68
+P 6300 1100
+F 0 "#PWR0124" H 6300 950 50  0001 C CNN
+F 1 "+3.3V" H 6315 1273 50  0000 C CNN
+F 2 "" H 6300 1100 50  0001 C CNN
+F 3 "" H 6300 1100 50  0001 C CNN
+	1    6300 1100
+	1    0    0    -1
+$EndComp
+Wire Wire Line
+	6000 1150 6300 1150
+Wire Wire Line
+	6300 1150 6300 1100
+Wire Wire Line
+	6800 2350 6800 2500
+Wire Wire Line
+	6800 2500 7050 2500
+Wire Wire Line
+	6200 2350 6800 2350
+Wire Wire Line
+	6700 2550 6700 2650
+Wire Wire Line
+	6700 2650 7050 2650
+Wire Wire Line
+	6300 2550 6700 2550
+$Sheet
+S 7050 3450 900  900
+U 5DEF398F
+F0 "SSM3302_2" 50
+F1 "SSM3302.sch" 50
+F2 "IN_L" I L 7050 3750 50
+F3 "IN_R" I L 7050 3600 50
+$EndSheet
+Wire Wire Line
+	6650 2700 6650 3600
+Wire Wire Line
+	6650 3600 7050 3600
+Wire Wire Line
+	4950 2700 6650 2700
+Wire Wire Line
+	6550 2900 6550 3750
+Wire Wire Line
+	6550 3750 7050 3750
+Wire Wire Line
+	5900 2900 6550 2900
+$Sheet
+S 1300 4200 500  450
+U 5DD36E4D
+F0 "EEPROM" 50
+F1 "EEPROM.sch" 50
+F2 "WP" I L 1300 4550 50
+F3 "SCL" I L 1300 4350 50
+F4 "SDA" I L 1300 4450 50
+$EndSheet
+Wire Wire Line
+	1200 4000 1200 4350
+Wire Wire Line
+	1200 4350 1300 4350
+Wire Wire Line
+	1100 3900 1100 4450
+Wire Wire Line
+	1100 4450 1300 4450
+Wire Wire Line
+	1000 3800 1000 4550
+Wire Wire Line
+	1000 4550 1300 4550
+$Comp
+L Connector:Conn_01x02_Female J8
+U 1 1 5DD615F2
+P 700 4000
+F 0 "J8" H 592 3675 50  0000 C CNN
+F 1 "CONN_EEPROM" H 592 3766 50  0000 C CNN
+F 2 "Connector_PinHeader_2.54mm:PinHeader_1x02_P2.54mm_Vertical" H 700 4000 50  0001 C CNN
+F 3 "~" H 700 4000 50  0001 C CNN
+	1    700  4000
+	-1   0    0    1
+$EndComp
+Wire Wire Line
+	1200 4000 900  4000
+Wire Wire Line
+	1100 3900 900  3900
+Wire Wire Line
+	1000 3800 2600 3800
+Wire Wire Line
+	1100 3900 2600 3900
+Connection ~ 1100 3900
+Wire Wire Line
+	2600 4000 1200 4000
+Connection ~ 1200 4000
 $EndSCHEMATC

Commit message: done
Parts:
- removed J1: MP 0-2, 691213710003:691213710003, symbol Connector:Conn_01x03_Male
- removed J2: Audio In, 691213710003:691213710003, symbol Connector:Conn_01x03_Male
- removed J3: MP 3-5, 691213710003:691213710003, symbol Connector:Conn_01x03_Male
- removed J4: MP 6-8, 691213710003:691213710003, symbol Connector:Conn_01x03_Male
- removed J5: MP 9-11, 691213710003:691213710003, symbol Connector:Conn_01x03_Male
- removed J6: Power Connector, 691213710003:691213710003, symbol Connector:Conn_01x03_Male
- removed J7: Audio Out (Headphones), 691213710003:691213710003, symbol Connector:Conn_01x03_Male
- added C46: 56nF, Capacitor_SMD:C_0805_2012Metric_Pad1.15x1.40mm_HandSolder, symbol Device:C_Small
- added C47: 3n3F, Capacitor_SMD:C_0805_2012Metric_Pad1.15x1.40mm_HandSolder, symbol Device:C_Small
- added C48, C50, C52: 100nF, Capacitor_SMD:C_0805_2012Metric_Pad1.15x1.40mm_HandSolder, symbol Device:C_Small
- added C49, C51: 10uF, Capacitor_SMD:C_0805_2012Metric_Pad1.15x1.40mm_HandSolder, symbol Device:C_Small
- added C53: 47uF, Capacitor_SMD:C_0805_2012Metric_Pad1.15x1.40mm_HandSolder, symbol Device:C_Small
- added J1, J2, J4: Conn_01x03_Female, 691213710003:691213710003, symbol Connector:Conn_01x03_Female
- added J10: NOT_PWR_CONN, Connector_PinHeader_2.54mm:PinHeader_1x01_P2.54mm_Vertical, symbol Connector:Conn_01x01_Male
- added J11: 3.3V_Conn, Connector_PinHeader_2.54mm:PinHeader_1x01_P2.54mm_Vertical, symbol Connector:Conn_01x01_Male
- added J12: GND_Conn, Connector_PinHeader_2.54mm:PinHeader_1x01_P2.54mm_Vertical, symbol Connector:Conn_01x01_Male
- added J13: 5V_Conn, Connector_PinHeader_2.54mm:PinHeader_1x01_P2.54mm_Vertical, symbol Connector:Conn_01x01_Male
- added J18: WB_Pin, Connector_PinHeader_2.54mm:PinHeader_1x01_P2.54mm_Vertical, symbol Connector:Conn_01x01_Male
- added J19: Reset, Connector_PinHeader_2.54mm:PinHeader_1x01_P2.54mm_Vertical, symbol Connector:Conn_01x01_Male
- added J3: Conn_01x12_Female, Connector_PinHeader_2.54mm:PinHeader_1x12_P2.54mm_Vertical, symbol Connector:Conn_01x12_Female
- added R23: 475r, Resistor_SMD:R_0805_2012Metric_Pad1.15x1.40mm_HandSolder, symbol Device:R_Small_US
Connections:
- net labels added: +5V, NOT_PWR
- wire segments 95 -> 150
