File: Board/EEPROM.sch (KiCad schematic (older format))
At the start: 3 parts, among them U5 CAT24C16WI-GT3

Commit message: done
Parts:
- removed U5: CAT24C16WI-GT3, CAT24 EEPROM:CAT24C16WI-GT3, symbol CAT24C16WIGT3:CAT24C16WI-GT3
- added U5: CAT24C16WI-GT3, CAT24:CAT24C16WI-GT3, symbol CAT24:CAT24C16WI-GT3
Connections:
- net +3V3: now also U5.8 (VCC)
- net GND: now also U5.4 (VSS)
- net SCL: now also U5.6 (SCL)
- net SDA: now also U5.5 (SDA)
- net WP: now also U5.7 (WP)
Changed lines of the file:
@@
 $EndDescr
-$Comp
-L CAT24C16WIGT3:CAT24C16WI-GT3 U?
-U 1 1 5DD38BFB
-P 3400 3350
-AR Path="/5DD38BFB" Ref="U?"  Part="1"
-AR Path="/5DD36E4D/5DD38BFB" Ref="U5"  Part="1"
-F 0 "U5" H 4200 3737 60  0000 C CNN
-F 1 "CAT24C16WI-GT3" H 4200 3631 60  0000 C CNN
-F 2 "CAT24 EEPROM:CAT24C16WI-GT3" H 4200 3590 60  0001 C CNN
-F 3 "" H 3400 3350 60  0000 C CNN
-	1    3400 3350
-	1    0    0    -1
-$EndComp
 $Comp
 L power:GND #PWR0133
@@
 Wire Wire Line
 	5850 3350 5850 3650
+$Comp
+L CAT24:CAT24C16WI-GT3 U5
+U 1 1 5DDE008D
+P 3400 3350
+F 0 "U5" H 4200 3737 60  0000 C CNN
+F 1 "CAT24C16WI-GT3" H 4200 3631 60  0000 C CNN
+F 2 "CAT24:CAT24C16WI-GT3" H 4200 3590 60  0001 C CNN
+F 3 "" H 3400 3350 60  0000 C CNN
+	1    3400 3350
+	1    0    0    -1
+$EndComp
 $EndSCHEMATC
