File: Board/SSM3302.sch (KiCad schematic (older format))
At the start: 5 parts, among them U2 SSM3302ACPZ-R7

Commit message: did some more stuff
Parts:
- removed U2: SSM3302ACPZ-R7, QFN50P600X600X80-41N, symbol SSM3302ACPZ-R7:SSM3302ACPZ-R7
- added C37, C38: 100nF, Capacitor_SMD:C_0805_2012Metric_Pad1.15x1.40mm_HandSolder, symbol Device:C_Small
- added R18, R19: 13k, Resistor_SMD:R_0805_2012Metric_Pad1.15x1.40mm_HandSolder, symbol Device:R_Small_US
- added U2: SSM3302ACPZ-R7, SSM3302:SSM3302ACPZ-R7, symbol 2019-11-17_04-12-08:SSM3302ACPZ-R7
- C20: value C_Small -> 470uF; footprint (none) -> Capacitor_SMD:C_0805_2012Metric_Pad1.15x1.40mm_HandSolder
- C21: value C_Small -> 10uF; footprint (none) -> Capacitor_SMD:C_0805_2012Metric_Pad1.15x1.40mm_HandSolder
- C22, C23: value C_Small -> 1uF; footprint (none) -> Capacitor_SMD:C_0805_2012Metric_Pad1.15x1.40mm_HandSolder
Connections:
- net +12V: now also U2.34 (PVDD), U2.35 (PVDD), U2.36 (PVDD), U2.37 (PVDD)
- net GND: now also C37.2, C38.2, U2.31 (PGND), U2.32 (PGND), U2.33 (PGND), U2.38 (PGND), U2.39 (PGND), U2.40 (PGND)
- new net: C37.1, R18.2
- new net: R18.1, U2.12 (INL-)
- new net: C38.1, R19.2
- new net: R19.1, U2.19 (INR-)
- new net IN_L: U2.11 (INL+)
- new net IN_R: U2.20 (INR+)
Other:
- moved on the sheet: C20, C21, C22, C23

Commit message: done
Parts:
- removed U2: SSM3302ACPZ-R7, SSM3302:SSM3302ACPZ-R7, symbol 2019-11-17_04-12-08:SSM3302ACPZ-R7
- added C39, C40, C41, C6: .22uF, Capacitor_SMD:C_0805_2012Metric_Pad1.15x1.40mm_HandSolder, symbol Device:C_Small
- added J14: THERM, Connector_PinHeader_2.54mm:PinHeader_1x01_P2.54mm_Vertical, symbol Connector:Conn_01x01_Male
- added J15: Gain_Conn, Connector_PinHeader_2.54mm:PinHeader_1x01_P2.54mm_Vertical, symbol Connector:Conn_01x01_Male
- added J5, J6: Conn_01x03_Female, 691213710003:691213710003, symbol Connector:Conn_01x03_Female
- added U2: SSM3302ACPZ-R7, SSM3302:SSM3302ACPZ-R7, symbol SSM3302:SSM3302ACPZ-R7
Connections:
- net +12V: now also U2.34 (PVDD), U2.35 (PVDD), U2.36 (PVDD), U2.37 (PVDD)
- net GND: now also U2.14 (TEST), U2.15 (TEST), U2.16 (MONO), U2.24 (AGND), U2.31 (PGND), U2.32 (PGND), U2.33 (PGND), U2.38 (PGND), U2.39 (PGND), U2.40 (PGND), U2.7 (AGND), U2.HTAB (EPAD)
- net IN_L: now also U2.11 (INL+)
- net IN_R: now also U2.20 (INR+)
- net at R18.1: now also U2.12 (INL-)
- net at R19.1: now also U2.19 (INR-)
- new net: C6.1, U2.1 (BOOTL+)
- new net: J14.1 (Pin_1), U2.17 (THERM)
- new net: C6.2, J5.2 (Pin_2), J5.3 (Pin_3), U2.2 (OUTL+), U2.3 (OUTL+)
- new net: J15.1 (Pin_1), U2.21 (GAIN)
- new net: C41.2, U2.25 (BOOTR-)
- new net: C41.1, J6.3 (Pin_3), U2.26 (OUTR-), U2.27 (OUTR-)
- new net: C40.1, J6.1 (Pin_1), J6.2 (Pin_2), U2.28 (OUTR+), U2.29 (OUTR+)
- new net: C40.2, U2.30 (BOOTR+)
- new net: C39.2, J5.1 (Pin_1), U2.4 (OUTL-), U2.5 (OUTL-)
- new net: C39.1, U2.6 (BOOTL-)
- new net +3V3: U2.23 (REGEN)
- new net +5V: U2.10 (EDGE), U2.8 (VREG/AVDD)
- new net NOT_PWR: U2.22 (*SDNR), U2.9 (*SDNL)
