File: Board/_autosave-Board.kicad_pcb (KiCad board)
At the start: 2 copper layers, 100 x 100 mm, 75 parts, among them J1 MP 0-2, J2 Audio In, J3 MP 3-5, J4 MP 6-8, J5 MP 9-11, J6 Power Connector, J7 Audio Out (Headphones), J8 CONN_EEPROM, Q1 Q_PNP_BCEC, U1 ADAU1701, U2 SSM3302ACPZ-R7, U3 ADP3336ARMZ, U4 SSM3302ACPZ-R7, U5 CAT24C16WI-GT3, Y1 Crystal_Small

Commit message: done
Parts:
- added C39: .22uF, Capacitor_SMD:C_0805_2012Metric_Pad1.15x1.40mm_HandSolder, F.Cu at (105.2, -52.9)
- added C40: .22uF, Capacitor_SMD:C_0805_2012Metric_Pad1.15x1.40mm_HandSolder, F.Cu at (109.9, -50.0)
- added C41: .22uF, Capacitor_SMD:C_0805_2012Metric_Pad1.15x1.40mm_HandSolder, F.Cu at (114.7, -55.4)
- added C42: .22uF, Capacitor_SMD:C_0805_2012Metric_Pad1.15x1.40mm_HandSolder, F.Cu at (167.7, -83.5)
- added C43: .22uF, Capacitor_SMD:C_0805_2012Metric_Pad1.15x1.40mm_HandSolder, F.Cu at (180.8, -97.8)
- added C44: .22uF, Capacitor_SMD:C_0805_2012Metric_Pad1.15x1.40mm_HandSolder, F.Cu at (176.1, -94.8)
- added C45: .22uF, Capacitor_SMD:C_0805_2012Metric_Pad1.15x1.40mm_HandSolder, F.Cu at (172.5, -83.5)
- added C46: 56nF, Capacitor_SMD:C_0805_2012Metric_Pad1.15x1.40mm_HandSolder, F.Cu at (102.0, -78.0)
- added C47: 3n3F, Capacitor_SMD:C_0805_2012Metric_Pad1.15x1.40mm_HandSolder, F.Cu at (92.6, -67.8)
- added C48: 100nF, Capacitor_SMD:C_0805_2012Metric_Pad1.15x1.40mm_HandSolder, F.Cu at (97.4, -72.0)
- added C49: 10uF, Capacitor_SMD:C_0805_2012Metric_Pad1.15x1.40mm_HandSolder, F.Cu at (127.0, -97.8)
- added C50: 100nF, Capacitor_SMD:C_0805_2012Metric_Pad1.15x1.40mm_HandSolder, F.Cu at (106.8, -76.5)
- added C51: 10uF, Capacitor_SMD:C_0805_2012Metric_Pad1.15x1.40mm_HandSolder, F.Cu at (97.3, -78.0)
- added C52: 100nF, Capacitor_SMD:C_0805_2012Metric_Pad1.15x1.40mm_HandSolder, F.Cu at (97.3, -75.0)
- added C53: 47uF, Capacitor_SMD:C_0805_2012Metric_Pad1.15x1.40mm_HandSolder, F.Cu at (92.6, -70.8)
- added C6: .22uF, Capacitor_SMD:C_0805_2012Metric_Pad1.15x1.40mm_HandSolder, F.Cu at (105.2, -47.0)
- added J10: NOT_PWR_CONN, Connector_PinHeader_2.54mm:PinHeader_1x01_P2.54mm_Vertical, F.Cu at (127.0, -91.0)
- added J11: 3.3V_Conn, Connector_PinHeader_2.54mm:PinHeader_1x01_P2.54mm_Vertical, F.Cu at (121.1, -87.0)
- added J12: GND_Conn, Connector_PinHeader_2.54mm:PinHeader_1x01_P2.54mm_Vertical, F.Cu at (106.8, -72.7)
- added J13: 5V_Conn, Connector_PinHeader_2.54mm:PinHeader_1x01_P2.54mm_Vertical, F.Cu at (111.5, -75.7)
- added J14: THERM, Connector_PinHeader_2.54mm:PinHeader_1x01_P2.54mm_Vertical, F.Cu at (119.4, -54.5)
- added J15: Gain_Conn, Connector_PinHeader_2.54mm:PinHeader_1x01_P2.54mm_Vertical, F.Cu at (114.6, -51.6)
- added J16: THERM, Connector_PinHeader_2.54mm:PinHeader_1x01_P2.54mm_Vertical, F.Cu at (181.9, -91.0)
- added J17: Gain_Conn, Connector_PinHeader_2.54mm:PinHeader_1x01_P2.54mm_Vertical, F.Cu at (177.2, -88.1)
- added J18: WB_Pin, Connector_PinHeader_2.54mm:PinHeader_1x01_P2.54mm_Vertical, F.Cu at (131.8, -96.9)
- added J19: Reset, Connector_PinHeader_2.54mm:PinHeader_1x01_P2.54mm_Vertical, F.Cu at (102.1, -68.2)
- added J9: Conn_01x03_Female, 691213710003:691213710003, F.Cu at (157.0, -94.3)
- added R23: 475r, Resistor_SMD:R_0805_2012Metric_Pad1.15x1.40mm_HandSolder, F.Cu at (102.0, -75.0)
- J1: value MP 0-2 -> Conn_01x03_Female
- J2: value Audio In -> Conn_01x03_Female
- J3: value MP 3-5 -> Conn_01x12_Female; footprint 691213710003:691213710003 -> Connector_PinHeader_2.54mm:PinHeader_1x12_P2.54mm_Vertical
- J4: value MP 6-8 -> Conn_01x03_Female
- J5: value MP 9-11 -> Conn_01x03_Female
- J6: value Power Connector -> Conn_01x03_Female
- J7: value Audio Out (Headphones) -> Conn_01x03_Female
- S1: footprint Switch:JS202011SCQN -> Switch JS202011SCQN:SW_JS202011SCQN
- U5: footprint CAT24 EEPROM:CAT24C16WI-GT3 -> CAT24:CAT24C16WI-GT3
- moved R5 189.4 mm to (141.8, -52.5)
- moved R22 184.4 mm to (160.6, -74.2)
- moved S1 184.2 mm to (153.2, -71.2)
- moved C10 180.9 mm to (142.2, -58.4)
- moved C8 180.9 mm to (142.2, -55.4)
- moved R18 179.9 mm to (172.5, -86.5)
- moved C9 177.7 mm to (137.1, -52.5)
- moved C34 176.9 mm to (137.4, -61.3)
- moved Q1 176.9 mm to (130.1, -58.6)
- moved C5 176.7 mm to (142.2, -61.3)
- moved C38 176.0 mm to (180.8, -94.8)
- moved J7 175.4 mm to (157.0, -84.4)
- moved R10 175.1 mm to (157.2, -57.1)
- moved C7 174.6 mm to (137.4, -55.4)
- moved U4 174.4 mm to (169.5, -95.1)
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Connections:
- J1 pad 1: Net-(J1-Pad1) -> GND
- J2 pad 1: Net-(J2-Pad1) -> GND
- J2 pad 2: Net-(J2-Pad2) -> GND
- J2 pad 3: Net-(J2-Pad3) -> +12V
- J4 pad 1: Net-(J4-Pad1) -> /SSM3302_1/IN_R
- J4 pad 2: Net-(J4-Pad2) -> /SSM3302_1/IN_L
- J4 pad 3: Net-(J4-Pad3) -> GND
- J5 pad 1: Net-(J5-Pad1) -> Net-(C39-Pad2)
- J5 pad 2: Net-(J5-Pad2) -> Net-(C6-Pad2)
- J5 pad 3: Net-(J5-Pad3) -> Net-(C6-Pad2)
- J6 pad 1: GND -> Net-(C40-Pad1)
- J6 pad 2: GND -> Net-(C40-Pad1)
- J6 pad 3: +12V -> Net-(C41-Pad1)
- J7 pad 1: /SSM3302_1/IN_R -> Net-(C43-Pad2)
- J7 pad 2: /SSM3302_1/IN_L -> Net-(C42-Pad2)
- J7 pad 3: GND -> Net-(C42-Pad2)
- R2 pad 2: Net-(R2-Pad2) -> Net-(J1-Pad3)
- R3 pad 2: Net-(R3-Pad2) -> Net-(J1-Pad2)
- U1 pad 10: Net-(J1-Pad2) -> Net-(J3-Pad2)
- U1 pad 11: Net-(J1-Pad1) -> Net-(J3-Pad1)
- U1 pad 14: Net-(J4-Pad2) -> Net-(J3-Pad8)
- U1 pad 15: Net-(J4-Pad1) -> Net-(J3-Pad7)
- U1 pad 16: Net-(J5-Pad2) -> Net-(J3-Pad11)
- U1 pad 19: Net-(J5-Pad3) -> Net-(J3-Pad12)
- U1 pad 26: Net-(J5-Pad1) -> Net-(J3-Pad10)
- U1 pad 27: Net-(J4-Pad3) -> Net-(J3-Pad9)
- U1 pad 28: Net-(J3-Pad1) -> Net-(J3-Pad4)
- U1 pad 29: Net-(J1-Pad3) -> Net-(J3-Pad3)
- U1 pad 38: Net-(U1-Pad38) -> GND
- U1 pad 39: Net-(U1-Pad39) -> +3V3
- U1 pad 6: Net-(U1-Pad6) -> +3V3
- U1 pad 7: Net-(U1-Pad7) -> GND
- U1 pad 8: Net-(J3-Pad2) -> Net-(J3-Pad5)
- U1 pad 9: Net-(J3-Pad3) -> Net-(J3-Pad6)
- U2 pad 10: Net-(U2-Pad10) -> +5V
- U2 pad 11: Net-(R16-Pad1) -> /SSM3302_1/IN_L
- U2 pad 12: /SSM3302_1/IN_L -> Net-(R16-Pad1)
- U2 pad 14: Net-(U2-Pad14) -> GND
- U2 pad 15: Net-(U2-Pad15) -> GND
- U2 pad 16: Net-(U2-Pad16) -> GND
- U2 pad 2: Net-(U2-Pad2) -> Net-(C6-Pad2)
- U2 pad 22: Net-(U2-Pad22) -> NOT_PWR
- U2 pad 23: Net-(U2-Pad23) -> +3V3
- U2 pad 24: Net-(U2-Pad24) -> GND
- U2 pad 26: Net-(U2-Pad26) -> Net-(C41-Pad1)
- U2 pad 27: Net-(U2-Pad27) -> Net-(C41-Pad1)
- U2 pad 28: Net-(U2-Pad28) -> Net-(C40-Pad1)
- U2 pad 29: Net-(U2-Pad29) -> Net-(C40-Pad1)
- U2 pad 3: Net-(U2-Pad3) -> Net-(C6-Pad2)
- U2 pad 4: Net-(U2-Pad4) -> Net-(C39-Pad2)
- U2 pad 5: Net-(U2-Pad5) -> Net-(C39-Pad2)
- U2 pad 7: Net-(U2-Pad7) -> GND
- U2 pad 8: Net-(U2-Pad8) -> +5V
- U2 pad 9: Net-(U2-Pad9) -> NOT_PWR
- U2 pad HTAB: Net-(U2-PadHTAB) -> GND
- U4 pad 10: Net-(U4-Pad10) -> +5V
- U4 pad 11: Net-(R18-Pad1) -> /SSM3302_2/IN_L
- U4 pad 12: /SSM3302_2/IN_L -> Net-(R18-Pad1)
- U4 pad 14: Net-(U4-Pad14) -> GND
- U4 pad 15: Net-(U4-Pad15) -> GND
- U4 pad 16: Net-(U4-Pad16) -> GND
- U4 pad 2: Net-(U4-Pad2) -> Net-(C42-Pad2)
- U4 pad 22: Net-(U4-Pad22) -> NOT_PWR
- U4 pad 23: Net-(U4-Pad23) -> +3V3
- U4 pad 24: Net-(U4-Pad24) -> GND
- U4 pad 26: Net-(U4-Pad26) -> Net-(C45-Pad1)
- U4 pad 27: Net-(U4-Pad27) -> Net-(C45-Pad1)
- U4 pad 28: Net-(U4-Pad28) -> Net-(C44-Pad1)
- U4 pad 29: Net-(U4-Pad29) -> Net-(C44-Pad1)
- U4 pad 3: Net-(U4-Pad3) -> Net-(C42-Pad2)
- U4 pad 4: Net-(U4-Pad4) -> Net-(C43-Pad2)
- U4 pad 5: Net-(U4-Pad5) -> Net-(C43-Pad2)
- U4 pad 7: Net-(U4-Pad7) -> GND
- U4 pad 8: Net-(U4-Pad8) -> +5V
- U4 pad 9: Net-(U4-Pad9) -> NOT_PWR
- U4 pad HTAB: Net-(U4-PadHTAB) -> GND
