File: Board/switch.sch (KiCad schematic (older format))
At the start: 2 parts

Commit message: done
Parts:
- S1: footprint Switch:JS202011SCQN -> Switch JS202011SCQN:SW_JS202011SCQN
Changed lines of the file:
@@
 Wire Wire Line
 	4400 4700 5000 4700
-$Comp
-L JS202011SCQN:JS202011SCQN S?
-U 1 1 5DD4636C
-P 5000 4050
-AR Path="/5DD36E4D/5DD4636C" Ref="S?"  Part="1"
-AR Path="/5DD36E4D/5DD45146/5DD4636C" Ref="S1"  Part="1"
-F 0 "S1" H 5330 4096 50  0000 L CNN
-F 1 "JS202011SCQN" H 5330 4005 50  0000 L CNN
-F 2 "Switch:JS202011SCQN" H 5000 4050 50  0001 L BNN
-F 3 "JS202011SCQN" H 5000 4050 50  0001 L BNN
-F 4 "JS Series DPDT On-On Gull Wing Surface Mount Subminiature Slide Switch" H 5000 4050 50  0001 L BNN "Field4"
-F 5 "Unavailable" H 5000 4050 50  0001 L BNN "Field5"
-F 6 "None" H 5000 4050 50  0001 L BNN "Field6"
-F 7 "C&K" H 5000 4050 50  0001 L BNN "Field7"
-F 8 "None" H 5000 4050 50  0001 L BNN "Field8"
-	1    5000 4050
-	1    0    0    -1
-$EndComp
 Wire Wire Line
 	4600 3250 4600 3400
@@
 Wire Wire Line
 	4600 3250 4750 3250
+$Comp
+L JS202011SCQN:JS202011SCQN S1
+U 1 1 5DDE2D28
+P 5000 4050
+F 0 "S1" H 5700 4000 50  0000 L CNN
+F 1 "JS202011SCQN" H 5650 3850 50  0000 L CNN
+F 2 "Switch JS202011SCQN:SW_JS202011SCQN" H 5000 4050 50  0001 L BNN
+F 3 "JS202011SCQN" H 5000 4050 50  0001 L BNN
+F 4 "JS Series DPDT On-On Gull Wing Surface Mount Subminiature Slide Switch" H 5000 4050 50  0001 L BNN "Field4"
+F 5 "Unavailable" H 5000 4050 50  0001 L BNN "Field5"
+F 6 "None" H 5000 4050 50  0001 L BNN "Field6"
+F 7 "C&K" H 5000 4050 50  0001 L BNN "Field7"
+F 8 "None" H 5000 4050 50  0001 L BNN "Field8"
+	1    5000 4050
+	1    0    0    -1
+$EndComp
 $EndSCHEMATC
