File: DSP/Board.sch (KiCad schematic (older format))
At the start: 48 parts, among them J1 Conn_01x03_Female, J10 NOT_PWR_CONN, J11 3.3V_Conn, J12 GND_Conn, J18 WB_Pin, J19 Reset, J2 Conn_01x03_Female, J3 Conn_01x12_Female, J4 Conn_01x03_Female, J8 CONN_EEPROM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

Commit message: split
Parts:
- removed J10: NOT_PWR_CONN, Connector_PinHeader_2.54mm:PinHeader_1x01_P2.54mm_Vertical, symbol Connector:Conn_01x01_Male
- added J5: 12v_2, 691213710003:691213710003, symbol Connector:Conn_01x03_Female
- added J6: Out_23_2, WJ250A-3.50-2P:WJ250A3502P, symbol Connector:Conn_01x02_Female
- added J7: Out_01_2, WJ250A-3.50-2P:WJ250A3502P, symbol Connector:Conn_01x02_Female
- added J9: Out_23_1, 691213710003:691213710003, symbol Connector:Conn_01x03_Female
- J1: value Conn_01x03_Female -> Audio_in
- J2: value Conn_01x03_Female -> 12v_1
- J4: value Conn_01x03_Female -> Out_01_1
Connections:
- net labels removed: +5V
- wire segments 267 -> 268

Commit message: finished DSP and AMP
Parts:
- removed J1: Audio_in, 691213710003:691213710003, symbol Connector:Conn_01x03_Female
- removed J3: Conn_01x12_Female, Connector_PinHeader_2.54mm:PinHeader_1x12_P2.54mm_Vertical, symbol Connector:Conn_01x12_Female
- removed J4: Out_01_1, 691213710003:691213710003, symbol Connector:Conn_01x03_Female
- removed J5: 12v_2, 691213710003:691213710003, symbol Connector:Conn_01x03_Female
- removed J9: Out_23_1, 691213710003:691213710003, symbol Connector:Conn_01x03_Female
- removed S1: JS202011SCQN, Switch JS202011SCQN:SW_JS202011SCQN, symbol JS202011SCQN:JS202011SCQN
- added D1: LED, LED_SMD:LED_0805_2012Metric_Pad1.15x1.40mm_HandSolder, symbol Device:LED
- added J1, J4, J9: SJ1-3535N, SJ1-3535N:CUI_SJ1-3535N, symbol SJ1-3535N:SJ1-3535N
- added J10: Conn_01x03_Female, Connector_PinSocket_2.54mm:PinSocket_1x03_P2.54mm_Vertical, symbol Connector:Conn_01x03_Female
- added J13: IO_2, Connector_PinHeader_2.54mm:PinHeader_1x01_P2.54mm_Vertical, symbol Connector:Conn_01x01_Female
- added J14: IO_3, Connector_PinHeader_2.54mm:PinHeader_1x04_P2.54mm_Vertical, symbol Connector:Conn_01x04_Female
- added J15: PowerConn, Connector_PinHeader_2.54mm:PinHeader_1x02_P2.54mm_Vertical, symbol Connector:Conn_01x02_Female
- added J16, J17, J20: Conn_01x01_Female, MountingHole:MountingHole_3.2mm_M3_ISO7380_Pad, symbol Connector:Conn_01x01_Female
- added J3: IO_1, Connector_PinHeader_2.54mm:PinHeader_1x07_P2.54mm_Vertical, symbol Connector:Conn_01x07_Female
- added J5: USB_B_Micro, MicroUSB:C77238, symbol Connector:USB_B_Micro
- added R12: 100R, Resistor_SMD:R_0805_2012Metric_Pad1.15x1.40mm_HandSolder, symbol Device:R_Small_US
- U3: symbol CAT24:CAT24C16WI-GT3 -> Board-rescue:CAT24C16WI-GT3-CAT24
Connections:
- net +12V: now also J15.2 (Pin_2); no longer J2.3 (Pin_3)
- net +3V3: now also R12.1
- net GND: now also D1.1 (K), J1.1, J10.3 (Pin_3), J16.1 (Pin_1), J17.1 (Pin_1), J20.1 (Pin_1), J4.1, J5.5 (GND), J9.1
- net output filter  4/Out: now also J9.2, J9.4
- net output filter 1/Out: now also J4.3, J4.5
- net output filter 2/Out: now also J4.2, J4.4
- net output filter 3/Out: now also J9.3, J9.5
- net at U1.10 (MP1): now also J3.3 (Pin_3)
- net at U1.11 (MP0): now also J3.4 (Pin_4)
- net at U1.14 (MP7): now also J3.5 (Pin_5)
- net at U1.15 (MP6): now also J3.6 (Pin_6)
- net at U1.16 (MP10): now also J3.7 (Pin_7)
- net at U1.19 (MP11): now also J13.1 (Pin_1)
- net at U1.21 (CLATCH/WP), U3.7 (WP): now also J10.2 (Pin_2)
- net at U1.26 (MP9): now also J14.4 (Pin_4)
- net at U1.27 (MP8): now also J14.3 (Pin_3)
- net at U1.28 (MP3): now also J14.2 (Pin_2)
- net at U1.29 (MP2): now also J14.1 (Pin_1)
- net at U1.8 (MP4): now also J3.1 (Pin_1)
- net at U1.9 (MP5): now also J3.2 (Pin_2)
- net at R3.2: now also J1.2, J1.4
- net at R2.2: now also J1.3, J1.5
- net at R11.2: now also J10.1 (Pin_1)
- new net: J15.1 (Pin_1), J2.3 (Pin_3), J5.1 (VBUS)
- new net: D1.2 (A), R12.2
- no-connect marks 3 -> 4
Other:
- moved on the sheet: J11, J2
