File: DSP/backup.kicad_pcb (KiCad board)
At the start: 2 copper layers, 90 x 75 mm, 72 parts, among them J1 SJ1-3535N, J10 Conn_01x03_Female, J11 3.3V_Conn, J12 GND_Conn, J13 IO_2, J14 IO_3, J15 PowerConn, J16 Conn_01x01_Female, J17 Conn_01x01_Female, J18 WB_Pin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

Commit message: finished DSP and AMP
Parts:
- removed D1: LED, LED_SMD:LED_0805_2012Metric_Pad1.15x1.40mm_HandSolder
- removed G***: LOGO, logo:logo_7_5mm
- removed J15: PowerConn, Connector_PinHeader_2.54mm:PinHeader_1x02_P2.54mm_Vertical
- removed J16, J17, J20: Conn_01x01_Female, MountingHole:MountingHole_3.2mm_M3_ISO7380_Pad
- removed R12: 100R, Resistor_SMD:R_0805_2012Metric_Pad1.15x1.40mm_HandSolder
- J1: value SJ1-3535N -> Audio_in; footprint SJ1-3535N:CUI_SJ1-3535N -> 691213710003:691213710003
- J4: value SJ1-3535N -> Out_01_1; footprint SJ1-3535N:CUI_SJ1-3535N -> 691213710003:691213710003
- J5: value USB_B_Micro -> 12v_2; footprint MicroUSB:C77238 -> 691213710003:691213710003
- J9: value SJ1-3535N -> Out_23_1; footprint SJ1-3535N:CUI_SJ1-3535N -> 691213710003:691213710003
- moved J9 22.6 mm to (124.2, 95.4), turned to 180 degrees
- moved C19 14.4 mm to (117.2, 79.5), turned to 270 degrees
- moved J6 13.7 mm to (125.1, 86.1)
- moved C17 8.44 mm to (102.6, 79.6), turned to 270 degrees
- moved R9 8.26 mm to (112.3, 79.5), turned to 270 degrees
- moved J1 7.06 mm to (69.9, 101.4), turned to 90 degrees
- moved C18 6.99 mm to (112.3, 84.3), turned to 270 degrees
- moved J4 6.76 mm to (89.0, 79.5), turned to 0 degrees
- moved J5 5.38 mm to (141.5, 98.2)
- moved R8 4.71 mm to (107.5, 79.6), turned to 270 degrees
- moved J12 2.56 mm to (123.7, 104.1)
- moved R2 2.56 mm to (78.2, 96.3)
- moved R3 2.56 mm to (78.2, 101.4)
- moved C33 2.52 mm to (141.6, 112.4)
- moved J2 2.50 mm to (141.6, 81.5)
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Connections:
- J2 pad 3: Net-(J15-Pad1) -> +12V
- J4 pad 1: GND -> /output filter 1/Out
- J4 pad 3: /output filter 1/Out -> GND
- J5 pad 1: Net-(J15-Pad1) -> GND
- J5 pad 2: Net-(J5-Pad2) -> GND
- J5 pad 3: Net-(J5-Pad3) -> +12V
- J9 pad 1: GND -> /output filter 3/Out
- J9 pad 3: /output filter 3/Out -> GND
Routing:
- net /output filter  4/Out: track 61.7 -> 27.6 mm
- net Net-(J15-Pad1): track 25.4 -> 0.00 mm
- net +12V: track 17.4 -> 34.7 mm
- net /output filter 3/Out: track 35.6 -> 49.8 mm
- net Net-(J1-Pad2): track 19.1 -> 7.23 mm
- net /output filter 2/Out: track 50.8 -> 39.9 mm
- net GND: track 113.1 -> 103.3 mm, vias 25 -> 22
- net +3V3: track 231.7 -> 240.7 mm
- net /output filter 1/Out: track 30.0 -> 23.8 mm
- net /output filter  4/In: track 29.8 -> 35.5 mm
- net Net-(J8-Pad2): track 58.0 -> 54.1 mm
- net Net-(J1-Pad3): track 10.9 -> 7.26 mm
- net Net-(D1-Pad2): track 3.40 -> 0.00 mm
- net /output filter 3/In: track 37.5 -> 35.0 mm
- net Net-(R3-Pad1): track 32.7 -> 35.0 mm
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- removed copper zone on F.Cu, net +12V
- removed copper zone on F.Cu, net +3V3
- removed copper zone on F.Cu, net /output filter  4/Out
- removed copper zone on F.Cu, net /output filter 1/Out
- removed copper zone on F.Cu, net /output filter 2/Out
- removed copper zone on F.Cu, net /output filter 3/Out
- removed copper zone on F.Cu, net GND
- removed copper zone on F.Cu, net Net-(J15-Pad1)
Other:
- outline, holes or cut-outs redrawn
- board text removed: "12/2019"
- board text removed: "12V"
- board text removed: "3V3"
- board text removed: "67.50 x 47.50 mm"
- board text removed: "90.00 x 75.00 mm"
- board text removed: "ADAU1701 Ben Xie"
- board text removed: "GND"
- board text removed: "MP0"
- board text removed: "MP1"
- board text removed: "MP10"
- board text removed: "MP11"
- board text removed: "MP2"
- board text removed: "MP3"
- board text removed: "MP4"
- board text removed: "MP5"
- board text removed: "MP6"
- board text removed: "MP7"
- board text removed: "MP8"
- board text removed: "MP9"
- board text removed: "RESET"
- board text removed: "SCL/ CCLK"
- board text removed: "SDA/ COUT"
- board text removed: "VO_0"
- board text removed: "VO_1"
- board text removed: "VO_2"
- board text removed: "VO_3"
- board text removed: "WB_Pin"
- board text removed: "WP"
